Commit message: Created new launch for kinova plus realsense

File: src/ros_kortex/kortex_description/arms/gen3/7dof/urdf/gen3_macro.xacro (robot description, xacro)
@@ -333,5 +333,5 @@
       <link name="${prefix}realsense_link" />
       <joint name="${prefix}realsense_module" type="fixed">
-        <origin xyz="0 0.05639 -0.00305" rpy="3.14159265358979 3.14159265358979 0" />
+        <origin xyz="0 0.035 -0.012" rpy="4.71238898038 4.71238898038 0" />
         <parent link="${prefix}end_effector_link" />
         <child  link="${prefix}realsense_link" />

File: src/ros_kortex/kortex_description/robots/kortex_robot.xacro (robot description, xacro)
@@ -35,4 +35,5 @@
         <xacro:if value="${realsense}">
             <xacro:sensor_d435 parent="${prefix}realsense_link">
+                <origin xyz="0 0 0" rpy="0 0 0"/>
             </xacro:sensor_d435>
         </xacro:if>
