Commit message: Changed Realsense box dimension to avoid collision in moveit

File: src/realsense2_description/urdf/_d435.urdf.xacro (robot description, xacro)
@@ -56,5 +56,6 @@
         <origin xyz="0 ${-d435_cam_depth_py} 0" rpy="0 0 0"/>
         <geometry>
-        <box size="${d435_cam_depth} ${d435_cam_width} ${d435_cam_height}"/>
+        <!-- <box size="${d435_cam_depth} ${d435_cam_width} ${d435_cam_height}"/> -->
+        <box size= "0.0001 0.0001 0.0001" />
         </geometry>
       </collision>
